Commit message: caibration and simulation

File: kuka_simulation/config/kuka_workcell.xacro (robot description, xacro)
@@ -3,5 +3,28 @@
     <!-- kuka macro -->
     <xacro:include filename="$(find kuka_simulation)/config/gazebo_kuka_kr6r700sixx.urdf" />
+    <!-- <xacro:include filename="$(find kuka_simulation)/config/camera.gazebo" /> -->
+    <xacro:property name="camera_link" value="0.05" /> <!-- Size of square 'camera' box -->
     <link name="world"/>
+    <!-- Camera -->
+    <link name="camera_link">
+        <collision>
+            <origin xyz="0 0 0" rpy="0 0 0"/>
+            <geometry>
+        <box size="${camera_link} ${camera_link} ${camera_link}"/>
+            </geometry>
+        </collision>
+        <visual>
+            <origin xyz="0 0 0" rpy="0 0 0"/>
+            <geometry>
+        <box size="${camera_link} ${camera_link} ${camera_link}"/>
+            </geometry>
+            <material name="red"/>
+        </visual>
+        <inertial>
+            <mass value="1e-5" />
+            <origin xyz="0 0 0" rpy="0 0 0"/>
+            <inertia ixx="1e-6" ixy="0" ixz="0" iyy="1e-6" iyz="0" izz="1e-6" />
+        </inertial>
+    </link>
     <!--mounting plate-->
     <link name="robot_mounting_plate">
@@ -145,4 +168,21 @@
             </geometry>
         </collision>
+    </link>
+    <joint name="camera_joint" type="fixed">
+        <axis xyz="0 1 0" />
+        <origin xyz="0.42 -0.82 0.62" rpy="0 0 0"/>
+        <parent link="world"/>
+        <child link="camera_link"/>
+    </joint>
+    <!-- generate an optical frame http://www.ros.org/reps/rep-0103.html#suffix-frames
+      so that ros and opencv can operate on the camera frame correctly -->
+    <joint name="camera_optical_joint" type="fixed">
+        <!-- these values have to be these values otherwise the gazebo camera image
+            won't be aligned properly with the frame it is supposedly originating from -->
+        <origin xyz="0 0 0" rpy="${-pi/2} 0 ${-pi/2}"/>
+        <parent link="camera_link"/>
+        <child link="camera_link_optical"/>
+    </joint>
+    <link name="camera_link_optical">
     </link>
     <joint name="robot_mounting_plate_top_to_world" type="fixed">

Commit message: Changed vision folder to have subfolders
Camera calibration now works and has been added to the simulation environment

Added pose estimation in 2d based on homography works to some extend

File: kuka_simulation/config/kuka_workcell.xacro (robot description, xacro)
@@ -4,5 +4,5 @@
     <xacro:include filename="$(find kuka_simulation)/config/gazebo_kuka_kr6r700sixx.urdf" />
     <!-- <xacro:include filename="$(find kuka_simulation)/config/camera.gazebo" /> -->
-    <xacro:property name="camera_link" value="0.05" /> <!-- Size of square 'camera' box -->
+    <xacro:property name="camera_link" value="0.03" /> <!-- Size of square 'camera' box -->
     <link name="world"/>
     <!-- Camera -->
@@ -11,5 +11,5 @@
             <origin xyz="0 0 0" rpy="0 0 0"/>
             <geometry>
-        <box size="${camera_link} ${camera_link} ${camera_link}"/>
+        <box size="0.06 ${camera_link} ${camera_link}"/>
             </geometry>
         </collision>
@@ -17,5 +17,5 @@
             <origin xyz="0 0 0" rpy="0 0 0"/>
             <geometry>
-        <box size="${camera_link} ${camera_link} ${camera_link}"/>
+        <box size="0.06 ${camera_link} ${camera_link}"/>
             </geometry>
             <material name="red"/>
@@ -171,5 +171,5 @@
     <joint name="camera_joint" type="fixed">
         <axis xyz="0 1 0" />
-        <origin xyz="0.42 -0.82 0.62" rpy="0 0 0"/>
+        <origin xyz="0.3859 -0.8837 0.5477" rpy="-2.5334 0.0440 -0.0288"/>
         <parent link="world"/>
         <child link="camera_link"/>
@@ -217,5 +217,5 @@
     </joint>
     <joint name="left_wall_ref_to_world" type="fixed">
-        <origin xyz="-0.916 -0.87 -0.881" rpy="0 0 0"/>
+        <origin xyz="-0.916 -0.92 -0.881" rpy="0 0 0"/>
         <parent link="world"/>
         <child link="left_wall_ref"/>

Commit message: Updated simulation workcell and other stuff, motion planning almost done

File: kuka_simulation/config/kuka_workcell.xacro (robot description, xacro)
@@ -6,4 +6,52 @@
     <xacro:property name="camera_link" value="0.03" /> <!-- Size of square 'camera' box -->
     <link name="world"/>
+    <!--Colors-->
+    <material name="black">
+        <color rgba="0.2 0.2 0.2 1.0"/>
+    </material>
+    <material name="gray">
+        <color rgba="0.9 0.9 0.9 1.0"/>
+    </material>
+    <material name="transparrent_gray">
+        <color rgba="0.9 0.9 0.9 0.5"/>
+    </material>
+    <material name="light_brown">
+        <color rgba="0.82 0.64 0.29 1.0"/>
+    </material>
+    <material name="red">
+        <color rgba="1.0 0.0 0.0 1.0"/>
+    </material>
+    <!-- actual TCP (virtual) -->
+    <link name="act_tcp"/>
+    <!--Gripper-->
+    <link name="gripper">
+        <visual>
+            <geometry>
+                <box size="0.089 0.049 0.063" />
+            </geometry>
+            <material name="gray"/>
+        </visual>
+        <collision>
+            <origin xyz="0 0 0" rpy="0 0 0" />
+            <geometry>
+                <box size="0.089 0.049 0.063" />
+            </geometry>
+        </collision>
+    </link>
+    <!--Gripping area-->
+    <link name="grasping_area">
+        <visual>
+            <geometry>
+                <box size="0.4 0.4 0.048" />
+            </geometry>
+            <material name="light_brown"/>
+        </visual>
+        <collision>
+            <origin xyz="0 0 0" rpy="0 0 0" />
+            <geometry>
+                <box size="0.4 0.4 0.048" />
+            </geometry>
+        </collision>
+    </link>
     <!-- Camera -->
     <link name="camera_link">
@@ -33,7 +81,5 @@
                 <box size="0.18 0.18 0.026" />
             </geometry>
-            <material name="light_gray">
-                <color rgba="0.5 0.9 0.9 1.0" />
-            </material>
+            <material name="black"/>
         </visual>
         <collision>
@@ -49,7 +95,5 @@
                 <box size="0.18 0.18 0.0" />
             </geometry>
-            <material name="light_gray">
-                <color rgba="0.5 0.9 0.9 1.0" />
-            </material>
+            <material name="black"/>
         </visual>
     </link>
@@ -60,7 +104,5 @@
                 <box size="2.0 0.5 0.855" />
             </geometry>
-            <material name="light_gray">
-                <color rgba="0.9 0.9 0.9 1.0" />
-            </material>
+            <material name="black"/>
         </visual>
         <collision>
@@ -76,7 +118,5 @@
                 <box size="0.0 0.0 0" />
             </geometry>
-            <material name="light_gray">
-                <color rgba="0.9 0.9 0.9 1.0" />
-            </material>
+            <material name="black"/>
         </visual>
     </link>
@@ -87,7 +127,5 @@
                 <box size="0.5 0.5 0.855" />
             </geometry>
-            <material name="light_gray">
-                <color rgba="0.9 0.9 0.9 1.0" />
-            </material>
+            <material name="black"/>
         </visual>
         <collision>
@@ -103,7 +141,5 @@
                 <box size="0.0 0.0 0" />
             </geometry>
-            <material name="light_gray">
-                <color rgba="0.9 0.9 0.9 1.0" />
-            </material>
+            <material name="black"/>
         </visual>
     </link>
@@ -114,7 +150,5 @@
                 <box size="2.75 0.01 2.10" />
             </geometry>
-            <material name="light_gray">
-                <color rgba="0.9 0.9 0.9 1.0" />
-            </material>
+            <material name="transparrent_gray"/>
         </visual>
         <collision>
@@ -130,7 +164,5 @@
                 <box size="0.0 0.0 0" />
             </geometry>
-            <material name="light_gray">
-                <color rgba="0.9 0.9 0.9 1.0" />
-            </material>
+            <material name="transparrent_gray"/>
         </visual>
     </link>
@@ -141,7 +173,5 @@
                 <box size="0.01 1.64 2.10" />
             </geometry>
-            <material name="light_gray">
-                <color rgba="0.9 0.9 0.9 1.0" />
-            </material>
+            <material name="transparrent_gray"/>
         </visual>
         <collision>
@@ -158,7 +188,5 @@
                 <box size="2.75 0.01 2.10" />
             </geometry>
-            <material name="light_gray">
-                <color rgba="0.9 0.9 0.9 1.0" />
-            </material>
+            <material name="transparrent_gray"/>
         </visual>
         <collision>
@@ -191,4 +219,20 @@
         <child link="robot_mounting_plate_top"/>
     </joint>
+    <joint name="flange_to_gripper" type="fixed">
+        <origin xyz="0.0445 0.0 0.0" rpy="0 0 0"/>
+        <parent link="flange"/>
+        <child link="gripper"/>
+    </joint>
+    <!--Set TCP postition-->
+    <joint name="tcp_to_robot" type="fixed">
+        <origin xyz="0 0 0.089" rpy="0 0 0"/>
+        <parent link="tool0"/>
+        <child link="act_tcp"/>
+    </joint>
+    <joint name="world_to_grasping_area" type="fixed">
+        <origin xyz="0.42903  -0.42587 -0.002" rpy="0 0 0"/>
+        <parent link="world"/>
+        <child link="grasping_area"/>
+    </joint>
     <joint name="robot_mounting_plate_to_robot_mounting_plate_top" type="fixed">
         <origin xyz="0 0 -0.013" rpy="0 0 0" />
